File: kewtea/kewtea.kicad_pcb (KiCad board)
At the start: 2 copper layers, 192 x 85 mm, 62 parts, among them J1 OLED_128x32, U1 Nice_Nano_V2

Commit message: removed dimensions and made zone fill smaller
Parts:
- D12: moved to B.Cu
